Commit message: skid-steer added

File: src/urdf/macros.xacro (robot description, xacro)
@@ -1,4 +1,5 @@
 <?xml version="1.0"?>
 <robot name="reckless_car" xmlns:xacro = "https://www.ros.org/wiki/xacro">
+<xacro:include filename="$(find exp_mini)/src/urdf/reckless_car.xacro" />
     <xacro:macro name='wheel_link' params='link_name'>
         <link name="${link_name}">
@@ -10,5 +11,5 @@
                 <origin xyz="0 0 0" rpy="1.570795 0 0"/>
                 <geometry>
-                    <cylinder radius="0.2" length="0.1"/>
+                    <cylinder radius="${wheelR}" length="$wheelT"/>
                 </geometry>
             </collision>
@@ -16,5 +17,5 @@
                 <origin xyz="0 0 0" rpy="1.570795 0 0"/>
                 <geometry>
-                    <cylinder radius="0.2" length="0.1"/>
+                    <cylinder radius="${wheelR}" length="$wheelT"/>
                 </geometry>
                 <material name="red"/>

File: src/urdf/reckless_car.xacro (robot description, xacro)
@@ -4,4 +4,6 @@
 <xacro:property name="baselw" value="1"/>
 <xacro:property name="baseh" value="0.25"/>
+<xacro:property name="wheelR" value="0.2"/>
+<xacro:property name="wheelT" value="0.25"/>
 <xacro:include filename="$(find exp_mini)/src/urdf/materials.xacro" />
 <xacro:include filename="$(find exp_mini)/src/urdf/macros.xacro" />
